Commit message: Improve formatting script, correctly align vectornav

File: urdf/sphere.urdf.xacro (robot description, xacro)
@@ -1,436 +1,436 @@
-<robot name="sphere">
-<link name="base_link">
-<visual>
-<origin xyz="0 0 0" rpy="0 -0 0" />
-<geometry>
-<mesh filename="package://sphere_description/meshes/lidar_imu_mount.stl"/>
-</geometry>
-<material name="lidar_imu_mount_material">
-<color rgba="0.90196078431372550543 0.90196078431372550543 0.90196078431372550543 1.0"/>
-</material>
-</visual>
-<collision>
-<origin xyz="0 0 0" rpy="0 -0 0" />
-<geometry>
-<mesh filename="package://sphere_description/meshes/lidar_imu_mount.stl"/>
-</geometry>
-</collision>
-<inertial>
-<origin xyz="0 0 0" rpy="0 0 0"/>
-<mass value="0" />
-<inertia ixx="0" ixy="0"  ixz="0" iyy="0" iyz="0" izz="0" />
-</inertial>
-</link>
-<link name="mti30_body">
-<visual>
-<origin xyz="-0.10027692321656977992 -0.038377640147504360479 -0.0068000000000000004885" rpy="0 -0 0" />
-<geometry>
-<mesh filename="package://sphere_description/meshes/mti30_body.stl"/>
-</geometry>
-<material name="mti30_body_material">
-<color rgba="0.72941176470588231506 0.35686274509803922461 0.023529411764705882026 1.0"/>
-</material>
-</visual>
-<collision>
-<origin xyz="-0.10027692321656977992 -0.038377640147504360479 -0.0068000000000000004885" rpy="0 -0 0" />
-<geometry>
-<mesh filename="package://sphere_description/meshes/mti30_body.stl"/>
-</geometry>
-</collision>
-<inertial>
-<origin xyz="0 0 0" rpy="0 0 0"/>
-<mass value="0" />
-<inertia ixx="0" ixy="0"  ixz="0" iyy="0" iyz="0" izz="0" />
-</inertial>
-</link>
-<link name="mti30">
-<inertial>
-<origin xyz="0 0 0" rpy="0 0 0" />
-<mass value="0" />
-<inertia ixx="0" ixy="0" ixz="0" iyy="0" iyz="0" izz="0" />
-</inertial>
-</link>
-<joint name="mti30_frame" type="fixed">
-<origin xyz="-0.030054161257389987172 0.0053761345939794813464 0.014306173174756259964" rpy="-7.8504622934188782988e-17 6.1629758220391558245e-32 2.3561944901923457252" />
-<parent link="mti30_body" />
-<child link="mti30" />
-<axis xyz="0 0 0"/>
-</joint>
-<joint name="mti30_base_joint" type="fixed">
-<origin xyz="0.075598896553159294909 0.013699613484093847715 0" rpy="3.141592653589793116 -0 -1.570796326794896558" />
-<parent link="base_link" />
-<child link="mti30_body" />
-<axis xyz="0 0 1"/>
-<limit effort="1" velocity="20" />
-<joint_properties friction="0.0"/>
-</joint>
-<link name="vn100_base">
-<visual>
-<origin xyz="-0.057102309884864574374 0.049250000000000009048 -0.0067999999999999996211" rpy="0 -0 0" />
-<geometry>
-<mesh filename="package://sphere_description/meshes/vn100_base.stl"/>
-</geometry>
-<material name="vn100_base_material">
-<color rgba="0.49803921568627451677 0.49803921568627451677 0.49803921568627451677 1.0"/>
-</material>
-</visual>
-<collision>
-<origin xyz="-0.057102309884864574374 0.049250000000000009048 -0.0067999999999999996211" rpy="0 -0 0" />
-<geometry>
-<mesh filename="package://sphere_description/meshes/vn100_base.stl"/>
-</geometry>
-</collision>
-<inertial>
-<origin xyz="0 0 0" rpy="0 0 0"/>
-<mass value="0" />
-<inertia ixx="0" ixy="0"  ixz="0" iyy="0" iyz="0" izz="0" />
-</inertial>
-</link>
-<link name="vn100_lid">
-<visual>
-<origin xyz="-0.065560509884864573427 0.039293200000000014227 -0.0096194000000000001727" rpy="0 -0 0" />
-<geometry>
-<mesh filename="package://sphere_description/meshes/vn100_lid.stl"/>
-</geometry>
-<material name="vn100_lid_material">
-<color rgba="0.86666666666666669627 0.32156862745098041545 0.15686274509803921351 1.0"/>
-</material>
-</visual>
-<collision>
-<origin xyz="-0.065560509884864573427 0.039293200000000014227 -0.0096194000000000001727" rpy="0 -0 0" />
-<geometry>
-<mesh filename="package://sphere_description/meshes/vn100_lid.stl"/>
-</geometry>
-</collision>
-<inertial>
-<origin xyz="0 0 0" rpy="0 0 0"/>
-<mass value="0" />
-<inertia ixx="0" ixy="0"  ixz="0" iyy="0" iyz="0" izz="0" />
-</inertial>
-</link>
-<link name="vn100">
-<inertial>
-<origin xyz="0 0 0" rpy="0 0 0" />
-<mass value="0" />
-<inertia ixx="0" ixy="0" ixz="0" iyy="0" iyz="0" izz="0" />
-</inertial>
-</link>
-<joint name="vn100_frame" type="fixed">
-<origin xyz="0.0069675361378467026707 -0.011647358283601402795 0.0011983999999999953023" rpy="3.141592653589793116 -0 -1.570796326794896558" />
-<parent link="vn100_lid" />
-<child link="vn100" />
-<axis xyz="0 0 0"/>
-</joint>
-<joint name="vectornav_lid_bottom_joint" type="fixed">
-<origin xyz="0.0084581999999999990525 0.0099567999999999948213 0.0038100000000000000186" rpy="0 -0 0" />
-<parent link="vn100_base" />
-<child link="vn100_lid" />
-<axis xyz="0 0 1"/>
-<limit effort="1" velocity="20" />
-<joint_properties friction="0.0"/>
-</joint>
-<joint name="vectornav_base_joint" type="fixed">
-<origin xyz="0.057102309884864574374 -0.049250000000000009048 0.0067999999999999996211" rpy="0 -0 0" />
-<parent link="base_link" />
-<child link="vn100_base" />
-<axis xyz="0 0 1"/>
-<limit effort="1" velocity="20" />
-<joint_properties friction="0.0"/>
-</joint>
-<link name="rslidar16_body">
-<visual>
-<origin xyz="-0.1881186521637837894 -0.068404028665133759235 -0.0006599999999999930575" rpy="-7.7037197775489434122e-34 -1.5407439555097886824e-33 1.9198621771937625091" />
-<geometry>
-<mesh filename="package://sphere_description/meshes/rslidar16_body.stl"/>
-</geometry>
-<material name="rslidar16_body_material">
-<color rgba="0.70196078431372543882 0.70196078431372543882 0.70196078431372543882 1.0"/>
-</material>
-</visual>
-<collision>
-<origin xyz="-0.1881186521637837894 -0.068404028665133759235 -0.0006599999999999930575" rpy="-7.7037197775489434122e-34 -1.5407439555097886824e-33 1.9198621771937625091" />
-<geometry>
-<mesh filename="package://sphere_description/meshes/rslidar16_body.stl"/>
-</geometry>
-</collision>
-<inertial>
-<origin xyz="0 0 0" rpy="0 0 0"/>
-<mass value="0" />
-<inertia ixx="0" ixy="0"  ixz="0" iyy="0" iyz="0" izz="0" />
-</inertial>
-</link>
-<link name="rslidar16">
-<inertial>
-<origin xyz="0 0 0" rpy="0 0 0" />
-<mass value="0" />
-<inertia ixx="0" ixy="0" ixz="0" iyy="0" iyz="0" izz="0" />
-</inertial>
-</link>
-<joint name="rslidar16_frame" type="fixed">
-<origin xyz="-1.3905711841025796972e-19 -2.3943233057370483929e-20 0.039799999999999995104" rpy="-3.8480234363252523323e-28 -8.7450794892603094459e-28 -3.141592653589793116" />
-<parent link="rslidar16_body" />
-<child link="rslidar16" />
-<axis xyz="0 0 0"/>
-</joint>
-<joint name="rslidar16_base_joint" type="fixed">
-<origin xyz="0 -1.4067523187999420031e-17 0.0067999999999999987538" rpy="-1.097024361507918903e-17 -9.4791237750517918037e-32 -0.34906585039886589561" />
-<parent link="base_link" />
-<child link="rslidar16_body" />
-<axis xyz="0 0 1"/>
-<limit effort="1" velocity="20" />
-<joint_properties friction="0.0"/>
-</joint>
-<link name="top_bottom_mount">
-<visual>
-<origin xyz="0.074999999999999983347 -5.4482878479313143175e-18 -0.0067999999999999727329" rpy="0 -0 0" />
-<geometry>
-<mesh filename="package://sphere_description/meshes/top_bottom_mount.stl"/>
-</geometry>
-<material name="top_bottom_mount_material">
-<color rgba="0.2313725490196078538 0.38039215686274507888 0.7058823529411765163 1.0"/>
-</material>
-</visual>
-<collision>
-<origin xyz="0.074999999999999983347 -5.4482878479313143175e-18 -0.0067999999999999727329" rpy="0 -0 0" />
-<geometry>
-<mesh filename="package://sphere_description/meshes/top_bottom_mount.stl"/>
-</geometry>
-</collision>
-<inertial>
-<origin xyz="0 0 0" rpy="0 0 0"/>
-<mass value="0" />
-<inertia ixx="0" ixy="0"  ixz="0" iyy="0" iyz="0" izz="0" />
-</inertial>
-</link>
-<link name="cover">
-<visual>
-<origin xyz="-0.016882738834749909385 -0.083659923351020154536 -0.061889999999999979752" rpy="-3.141592653589793116 -1.2246467991473529607e-16 2.7061648158250949834e-48" />
-<geometry>
-<mesh filename="package://sphere_description/meshes/cover.stl"/>
-</geometry>
-<material name="cover_material">
-<color rgba="0.61568627450980395466 0.81176470588235294379 0.92941176470588238168 1.0"/>
-</material>
-</visual>
-<collision>
-<origin xyz="-0.016882738834749909385 -0.083659923351020154536 -0.061889999999999979752" rpy="-3.141592653589793116 -1.2246467991473529607e-16 2.7061648158250949834e-48" />
-<geometry>
-<mesh filename="package://sphere_description/meshes/cover.stl"/>
-</geometry>
-</collision>
-<inertial>
-<origin xyz="0 0 0" rpy="0 0 0"/>
-<mass value="0" />
-<inertia ixx="0" ixy="0"  ixz="0" iyy="0" iyz="0" izz="0" />
-</inertial>
-</link>
-<link name="box">
-<visual>
-<origin xyz="0.076062912018315831375 0.024695847005800242169 -0.059502399999999969205" rpy="-3.141592653589793116 -1.2246467991473534537e-16 1.5637583885463270444e-47" />
-<geometry>
-<mesh filename="package://sphere_description/meshes/box.stl"/>
-</geometry>
-<material name="box_material">
-<color rgba="0.61568627450980395466 0.81176470588235294379 0.92941176470588238168 1.0"/>
-</material>
-</visual>
-<collision>
-<origin xyz="0.076062912018315831375 0.024695847005800242169 -0.059502399999999969205" rpy="-3.141592653589793116 -1.2246467991473534537e-16 1.5637583885463270444e-47" />
-<geometry>
-<mesh filename="package://sphere_description/meshes/box.stl"/>
-</geometry>
-</collision>
-<inertial>
-<origin xyz="0 0 0" rpy="0 0 0"/>
-<mass value="0" />
-<inertia ixx="0" ixy="0"  ixz="0" iyy="0" iyz="0" izz="0" />
-</inertial>
-</link>
-<link name="dps310">
-<inertial>
-<origin xyz="0 0 0" rpy="0 0 0" />
-<mass value="0" />
-<inertia ixx="0" ixy="0" ixz="0" iyy="0" iyz="0" izz="0" />
-</inertial>
-</link>
-<joint name="dps310_frame" type="fixed">
-<origin xyz="0.061019072575711902351 0.068023672350145891752 -0.018025099999999995293" rpy="-1.570796326794896558 1.2826107535319245424e-15 0.78539816339744805695" />
-<parent link="box" />
-<child link="dps310" />
-<axis xyz="0 0 0"/>
-</joint>
-<joint name="box_rpi_cover" type="fixed">
-<origin xyz="-0.092945650853065692187 -0.10835577035682041058 -0.0023876000000000036083" rpy="4.8985871965894128287e-16 -4.8985871965894118426e-16 -2.453048575909777067e-31" />
-<parent link="cover" />
-<child link="box" />
-<axis xyz="0 0 1"/>
-<limit effort="1" velocity="20" />
-<joint_properties friction="0.0"/>
-</joint>
-<joint name="box_rpi" type="fixed">
-<origin xyz="0.058009212746076954659 0.083767971770193142 -0.068689999999999959424" rpy="-3.1415926535897926719 3.673940397442058882e-16 -3.141592653589793116" />
-<parent link="top_bottom_mount" />
-<child link="cover" />
-<axis xyz="0 0 1"/>
-<limit effort="1" velocity="20" />
-<joint_properties friction="0.0"/>
-</joint>
-<link name="extrusions_bottom">
-<visual>
-<origin xyz="-1.2246467991473541932e-17 0.17999999999999999334 0.074670000000000000262" rpy="1.2246467991473534537e-16 -1.2246467991473534537e-16 -4.856562848648102935e-48" />
-<geometry>
-<mesh filename="package://sphere_description/meshes/extrusions_bottom.stl"/>
-</geometry>
-<material name="extrusions_bottom_material">
-<color rgba="0.75294117647058822484 0.75294117647058822484 0.75294117647058822484 1.0"/>
-</material>
-</visual>
-<collision>
-<origin xyz="-1.2246467991473541932e-17 0.17999999999999999334 0.074670000000000000262" rpy="1.2246467991473534537e-16 -1.2246467991473534537e-16 -4.856562848648102935e-48" />
-<geometry>
-<mesh filename="package://sphere_description/meshes/extrusions_bottom.stl"/>
-</geometry>
-</collision>
-<inertial>
-<origin xyz="0 0 0" rpy="0 0 0"/>
-<mass value="0" />
-<inertia ixx="0" ixy="0"  ixz="0" iyy="0" iyz="0" izz="0" />
-</inertial>
-</link>
-<link name="extrusions_top">
-<visual>
-<origin xyz="0.2000000000000000111 -0.20000000000000003886 0" rpy="3.141592653589793116 -0 1.5127223783572849212e-46" />
-<geometry>
-<mesh filename="package://sphere_description/meshes/extrusions_top.stl"/>
-</geometry>
-<material name="extrusions_top_material">
-<color rgba="0.75294117647058822484 0.75294117647058822484 0.75294117647058822484 1.0"/>
-</material>
-</visual>
-<collision>
-<origin xyz="0.2000000000000000111 -0.20000000000000003886 0" rpy="3.141592653589793116 -0 1.5127223783572849212e-46" />
-<geometry>
-<mesh filename="package://sphere_description/meshes/extrusions_top.stl"/>
-</geometry>
-</collision>
-<inertial>
-<origin xyz="0 0 0" rpy="0 0 0"/>
-<mass value="0" />
-<inertia ixx="0" ixy="0"  ixz="0" iyy="0" iyz="0" izz="0" />
-</inertial>
-</link>
-<joint name="extrusions_top" type="fixed">
-<origin xyz="-0.20000000000000003886 -0.020000000000000017764 0.074669999999999958629" rpy="-3.1415926535897922278 -8.5725275940314731898e-16 -8.0555926954094540157e-31" />
-<parent link="extrusions_bottom" />
-<child link="extrusions_top" />
-<axis xyz="0 0 1"/>
-<limit effort="1" velocity="20" />
-<joint_properties friction="0.0"/>
-</joint>
-<link name="eyebolt">
-<visual>
-<origin xyz="0 0 0" rpy="3.141592653589793116 -0 8.1822406464942546288e-47" />
-<geometry>
-<mesh filename="package://sphere_description/meshes/eyebolt.stl"/>
-</geometry>
-<material name="eyebolt_material">
-<color rgba="0.64705882352941179736 0.64705882352941179736 0.64705882352941179736 1.0"/>
-</material>
-</visual>
-<collision>
-<origin xyz="0 0 0" rpy="3.141592653589793116 -0 8.1822406464942546288e-47" />
-<geometry>
-<mesh filename="package://sphere_description/meshes/eyebolt.stl"/>
-</geometry>
-</collision>
-<inertial>
-<origin xyz="0 0 0" rpy="0 0 0"/>
-<mass value="0" />
-<inertia ixx="0" ixy="0"  ixz="0" iyy="0" iyz="0" izz="0" />
-</inertial>
-</link>
-<joint name="eyebolt" type="fixed">
-<origin xyz="2.6182847689831911583e-10 -0.019999999997707226806 -0.1253299999999999137" rpy="8.5725275940314731898e-16 8.5725275940314731898e-16 -1.570796326794896558" />
-<parent link="extrusions_bottom" />
-<child link="eyebolt" />
-<axis xyz="0 0 1"/>
-<limit effort="1" velocity="20" />
-<joint_properties friction="0.0"/>
-</joint>
-<link name="sheetmetal_2batteries_cover">
-<visual>
-<origin xyz="-0.0089900000000000101358 -1.3877787807814456755e-17 0.0089999999999999958505" rpy="-1.570796326794896336 -1.2246467991473532072e-16 0" />
-<geometry>
-<mesh filename="package://sphere_description/meshes/sheetmetal_2batteries_cover.stl"/>
-</geometry>
-<material name="sheetmetal_2batteries_cover_material">
-<color rgba="0.97254901960784312376 0.52941176470588235947 0.0039215686274509803377 1.0"/>
-</material>
-</visual>
-<collision>
-<origin xyz="-0.0089900000000000101358 -1.3877787807814456755e-17 0.0089999999999999958505" rpy="-1.570796326794896336 -1.2246467991473532072e-16 0" />
-<geometry>
-<mesh filename="package://sphere_description/meshes/sheetmetal_2batteries_cover.stl"/>
-</geometry>
-</collision>
-<inertial>
-<origin xyz="0 0 0" rpy="0 0 0"/>
-<mass value="0" />
-<inertia ixx="0" ixy="0"  ixz="0" iyy="0" iyz="0" izz="0" />
-</inertial>
-</link>
-<joint name="battery_box" type="fixed">
-<origin xyz="-0.010000000000000005412 -0.02581900000000000861 -2.7755575615628913511e-17" rpy="-1.570796326794896558 1.2246467991473534537e-16 -1.570796326794896558" />
-<parent link="extrusions_bottom" />
-<child link="sheetmetal_2batteries_cover" />
-<axis xyz="0 0 1"/>
-<limit effort="1" velocity="20" />
-<joint_properties friction="0.0"/>
-</joint>
-<joint name="extrusions_bottom" type="fixed">
-<origin xyz="0.094999999999999945599 -1.0906150302096335474e-17 -0.075329999999999938676" rpy="3.673940397442059375e-16 -3.673940397442059375e-16 -1.570796326794896558" />
-<parent link="top_bottom_mount" />
-<child link="extrusions_bottom" />
-<axis xyz="0 0 1"/>
-<limit effort="1" velocity="20" />
-<joint_properties friction="0.0"/>
-</joint>
-<link name="lidar_box">
-<visual>
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