Commit message: Fix xml formatting script

File: urdf/sphere.urdf.xacro (robot description, xacro)
@@ -2,14 +2,14 @@
 	<link name="base_link">
 		<visual>
-			<origin xyz="['0.0', '0.0', '0.0']" rpy="['0.0', '-0.0', '0.0']"/>
+			<origin xyz="0.0 0.0 0.0" rpy="0.0 -0.0 0.0"/>
 			<geometry>
 				<mesh filename="package://sphere_description/meshes/lidar_imu_mount.stl"/>
 			</geometry>
 			<material name="lidar_imu_mount_material">
-				<color rgba="['0.90196', '0.90196', '0.90196', '1.0']"/>
-			</material>
-		</visual>
-		<collision>
-			<origin xyz="['0.0', '0.0', '0.0']" rpy="['0.0', '-0.0', '0.0']"/>
+				<color rgba="0.90196 0.90196 0.90196 1.0"/>
+			</material>
+		</visual>
+		<collision>
+			<origin xyz="0.0 0.0 0.0" rpy="0.0 -0.0 0.0"/>
 			<geometry>
 				<mesh filename="package://sphere_description/meshes/lidar_imu_mount.stl"/>
@@ -17,5 +17,5 @@
 		</collision>
 		<inertial>
-			<origin xyz="['0.0', '0.0', '0.0']" rpy="['0.0', '0.0', '0.0']"/>
+			<origin xyz="0.0 0.0 0.0" rpy="0.0 0.0 0.0"/>
 			<mass value="0"/>
 			<inertia ixx="0" ixy="0" ixz="0" iyy="0" iyz="0" izz="0"/>
@@ -24,14 +24,14 @@
 	<link name="mti30_body">
 		<visual>
-			<origin xyz="['-0.10028', '-0.03838', '-0.0068']" rpy="['0.0', '-0.0', '0.0']"/>
+			<origin xyz="-0.10028 -0.03838 -0.0068" rpy="0.0 -0.0 0.0"/>
 			<geometry>
 				<mesh filename="package://sphere_description/meshes/mti30_body.stl"/>
 			</geometry>
 			<material name="mti30_body_material">
-				<color rgba="['0.72941', '0.35686', '0.02353', '1.0']"/>
-			</material>
-		</visual>
-		<collision>
-			<origin xyz="['-0.10028', '-0.03838', '-0.0068']" rpy="['0.0', '-0.0', '0.0']"/>
+				<color rgba="0.72941 0.35686 0.02353 1.0"/>
+			</material>
+		</visual>
+		<collision>
+			<origin xyz="-0.10028 -0.03838 -0.0068" rpy="0.0 -0.0 0.0"/>
 			<geometry>
 				<mesh filename="package://sphere_description/meshes/mti30_body.stl"/>
@@ -39,5 +39,5 @@
 		</collision>
 		<inertial>
-			<origin xyz="['0.0', '0.0', '0.0']" rpy="['0.0', '0.0', '0.0']"/>
+			<origin xyz="0.0 0.0 0.0" rpy="0.0 0.0 0.0"/>
 			<mass value="0"/>
 			<inertia ixx="0" ixy="0" ixz="0" iyy="0" iyz="0" izz="0"/>
@@ -46,5 +46,5 @@
 	<link name="mti30">
 		<inertial>
-			<origin xyz="['0.0', '0.0', '0.0']" rpy="['0.0', '0.0', '0.0']"/>
+			<origin xyz="0.0 0.0 0.0" rpy="0.0 0.0 0.0"/>
 			<mass value="0"/>
 			<inertia ixx="0" ixy="0" ixz="0" iyy="0" iyz="0" izz="0"/>
@@ -52,14 +52,14 @@
 	</link>
 	<joint name="mti30_frame" type="fixed">
-		<origin xyz="['-0.03005', '0.00538', '0.01431']" rpy="['-0.0', '-0.0', '0.7854']"/>
+		<origin xyz="-0.03005 0.00538 0.01431" rpy="-0.0 -0.0 0.7854"/>
 		<parent link="mti30_body"/>
 		<child link="mti30"/>
-		<axis xyz="['0.0', '0.0', '0.0']"/>
+		<axis xyz="0.0 0.0 0.0"/>
 	</joint>
 	<joint name="mti30_base_joint" type="fixed">
-		<origin xyz="['0.10028', '0.03838', '0.0068']" rpy="['0.0', '-0.0', '0.0']"/>
+		<origin xyz="0.10028 0.03838 0.0068" rpy="0.0 -0.0 0.0"/>
 		<parent link="base_link"/>
 		<child link="mti30_body"/>
-		<axis xyz="['0.0', '0.0', '1.0']"/>
+		<axis xyz="0.0 0.0 1.0"/>
 		<limit effort="1" velocity="20"/>
 		<joint_properties friction="0.0"/>
@@ -67,14 +67,14 @@
 	<link name="vn100_base">
 		<visual>
-			<origin xyz="['-0.0571', '0.04925', '-0.0068']" rpy="['0.0', '-0.0', '0.0']"/>
+			<origin xyz="-0.0571 0.04925 -0.0068" rpy="0.0 -0.0 0.0"/>
 			<geometry>
 				<mesh filename="package://sphere_description/meshes/vn100_base.stl"/>
 			</geometry>
 			<material name="vn100_base_material">
-				<color rgba="['0.49804', '0.49804', '0.49804', '1.0']"/>
-			</material>
-		</visual>
-		<collision>
-			<origin xyz="['-0.0571', '0.04925', '-0.0068']" rpy="['0.0', '-0.0', '0.0']"/>
+				<color rgba="0.49804 0.49804 0.49804 1.0"/>
+			</material>
+		</visual>
+		<collision>
+			<origin xyz="-0.0571 0.04925 -0.0068" rpy="0.0 -0.0 0.0"/>
 			<geometry>
 				<mesh filename="package://sphere_description/meshes/vn100_base.stl"/>
@@ -82,5 +82,5 @@
 		</collision>
 		<inertial>
-			<origin xyz="['0.0', '0.0', '0.0']" rpy="['0.0', '0.0', '0.0']"/>
+			<origin xyz="0.0 0.0 0.0" rpy="0.0 0.0 0.0"/>
 			<mass value="0"/>
 			<inertia ixx="0" ixy="0" ixz="0" iyy="0" iyz="0" izz="0"/>
@@ -89,14 +89,14 @@
 	<link name="vn100_lid">
 		<visual>
-			<origin xyz="['-0.06556', '0.03929', '-0.00962']" rpy="['0.0', '-0.0', '0.0']"/>
+			<origin xyz="-0.06556 0.03929 -0.00962" rpy="0.0 -0.0 0.0"/>
 			<geometry>
 				<mesh filename="package://sphere_description/meshes/vn100_lid.stl"/>
 			</geometry>
 			<material name="vn100_lid_material">
-				<color rgba="['0.86667', '0.32157', '0.15686', '1.0']"/>
-			</material>
-		</visual>
-		<collision>
-			<origin xyz="['-0.06556', '0.03929', '-0.00962']" rpy="['0.0', '-0.0', '0.0']"/>
+				<color rgba="0.86667 0.32157 0.15686 1.0"/>
+			</material>
+		</visual>
+		<collision>
+			<origin xyz="-0.06556 0.03929 -0.00962" rpy="0.0 -0.0 0.0"/>
 			<geometry>
 				<mesh filename="package://sphere_description/meshes/vn100_lid.stl"/>
@@ -104,5 +104,5 @@
 		</collision>
 		<inertial>
-			<origin xyz="['0.0', '0.0', '0.0']" rpy="['0.0', '0.0', '0.0']"/>
+			<origin xyz="0.0 0.0 0.0" rpy="0.0 0.0 0.0"/>
 			<mass value="0"/>
 			<inertia ixx="0" ixy="0" ixz="0" iyy="0" iyz="0" izz="0"/>
@@ -111,5 +111,5 @@
 	<link name="vn100">
 		<inertial>
-			<origin xyz="['0.0', '0.0', '0.0']" rpy="['0.0', '0.0', '0.0']"/>
+			<origin xyz="0.0 0.0 0.0" rpy="0.0 0.0 0.0"/>
 			<mass value="0"/>
 			<inertia ixx="0" ixy="0" ixz="0" iyy="0" iyz="0" izz="0"/>
@@ -117,22 +117,22 @@
 	</link>
 	<joint name="vn100_frame" type="fixed">
-		<origin xyz="['0.00697', '-0.01165', '0.0012']" rpy="['0.0', '-0.0', '1.5708']"/>
+		<origin xyz="0.00697 -0.01165 0.0012" rpy="0.0 -0.0 1.5708"/>
 		<parent link="vn100_lid"/>
 		<child link="vn100"/>
-		<axis xyz="['0.0', '0.0', '0.0']"/>
+		<axis xyz="0.0 0.0 0.0"/>
 	</joint>
 	<joint name="vectornav_lid_bottom_joint" type="fixed">
-		<origin xyz="['0.00846', '0.00996', '0.00381']" rpy="['0.0', '-0.0', '0.0']"/>
+		<origin xyz="0.00846 0.00996 0.00381" rpy="0.0 -0.0 0.0"/>
 		<parent link="vn100_base"/>
 		<child link="vn100_lid"/>
-		<axis xyz="['0.0', '0.0', '1.0']"/>
+		<axis xyz="0.0 0.0 1.0"/>
 		<limit effort="1" velocity="20"/>
 		<joint_properties friction="0.0"/>
 	</joint>
 	<joint name="vectornav_base_joint" type="fixed">
-		<origin xyz="['0.0571', '-0.04925', '0.0068']" rpy="['0.0', '-0.0', '0.0']"/>
+		<origin xyz="0.0571 -0.04925 0.0068" rpy="0.0 -0.0 0.0"/>
 		<parent link="base_link"/>
 		<child link="vn100_base"/>
-		<axis xyz="['0.0', '0.0', '1.0']"/>
+		<axis xyz="0.0 0.0 1.0"/>
 		<limit effort="1" velocity="20"/>
 		<joint_properties friction="0.0"/>
@@ -140,14 +140,14 @@
 	<link name="rslidar16_body">
 		<visual>
-			<origin xyz="['0.18812', '0.0684', '-0.00066']" rpy="['0.0', '-0.0', '-1.22173']"/>
+			<origin xyz="0.18812 0.0684 -0.00066" rpy="0.0 -0.0 -1.22173"/>
 			<geometry>
 				<mesh filename="package://sphere_description/meshes/rslidar16_body.stl"/>
 			</geometry>
 			<material name="rslidar16_body_material">
-				<color rgba="['0.70196', '0.70196', '0.70196', '1.0']"/>
-			</material>
-		</visual>
-		<collision>
-			<origin xyz="['0.18812', '0.0684', '-0.00066']" rpy="['0.0', '-0.0', '-1.22173']"/>
+				<color rgba="0.70196 0.70196 0.70196 1.0"/>
+			</material>
+		</visual>
+		<collision>
+			<origin xyz="0.18812 0.0684 -0.00066" rpy="0.0 -0.0 -1.22173"/>
 			<geometry>
 				<mesh filename="package://sphere_description/meshes/rslidar16_body.stl"/>
@@ -155,5 +155,5 @@
 		</collision>
 		<inertial>
-			<origin xyz="['0.0', '0.0', '0.0']" rpy="['0.0', '0.0', '0.0']"/>
+			<origin xyz="0.0 0.0 0.0" rpy="0.0 0.0 0.0"/>
 			<mass value="0"/>
 			<inertia ixx="0" ixy="0" ixz="0" iyy="0" iyz="0" izz="0"/>
@@ -162,5 +162,5 @@
 	<link name="rslidar16">
 		<inertial>
-			<origin xyz="['0.0', '0.0', '0.0']" rpy="['0.0', '0.0', '0.0']"/>
+			<origin xyz="0.0 0.0 0.0" rpy="0.0 0.0 0.0"/>
 			<mass value="0"/>
 			<inertia ixx="0" ixy="0" ixz="0" iyy="0" iyz="0" izz="0"/>
@@ -168,14 +168,14 @@
 	</link>
 	<joint name="rslidar16_frame" type="fixed">
-		<origin xyz="['0.0', '0.0', '0.0398']" rpy="['0.0', '0.0', '0.0']"/>
+		<origin xyz="0.0 0.0 0.0398" rpy="0.0 0.0 0.0"/>
 		<parent link="rslidar16_body"/>
 		<child link="rslidar16"/>
-		<axis xyz="['0.0', '0.0', '0.0']"/>
+		<axis xyz="0.0 0.0 0.0"/>
 	</joint>
 	<joint name="rslidar16_base_joint" type="fixed">
-		<origin xyz="['0.0', '-0.0', '0.0068']" rpy="['-0.0', '-0.0', '2.79253']"/>
+		<origin xyz="0.0 -0.0 0.0068" rpy="-0.0 -0.0 2.79253"/>
 		<parent link="base_link"/>
 		<child link="rslidar16_body"/>
-		<axis xyz="['0.0', '0.0', '1.0']"/>
+		<axis xyz="0.0 0.0 1.0"/>
 		<limit effort="1" velocity="20"/>
 		<joint_properties friction="0.0"/>
@@ -183,14 +183,14 @@
 	<link name="top_bottom_mount">
 		<visual>
-			<origin xyz="['0.075', '-0.0', '-0.0068']" rpy="['0.0', '-0.0', '0.0']"/>
+			<origin xyz="0.075 -0.0 -0.0068" rpy="0.0 -0.0 0.0"/>
 			<geometry>
 				<mesh filename="package://sphere_description/meshes/top_bottom_mount.stl"/>
 			</geometry>
 			<material name="top_bottom_mount_material">
-				<color rgba="['0.23137', '0.38039', '0.70588', '1.0']"/>
-			</material>
-		</visual>
-		<collision>
-			<origin xyz="['0.075', '-0.0', '-0.0068']" rpy="['0.0', '-0.0', '0.0']"/>
+				<color rgba="0.23137 0.38039 0.70588 1.0"/>
+			</material>
+		</visual>
+		<collision>
+			<origin xyz="0.075 -0.0 -0.0068" rpy="0.0 -0.0 0.0"/>
 			<geometry>
 				<mesh filename="package://sphere_description/meshes/top_bottom_mount.stl"/>
@@ -198,5 +198,5 @@
 		</collision>
 		<inertial>
-			<origin xyz="['0.0', '0.0', '0.0']" rpy="['0.0', '0.0', '0.0']"/>
+			<origin xyz="0.0 0.0 0.0" rpy="0.0 0.0 0.0"/>
 			<mass value="0"/>
 			<inertia ixx="0" ixy="0" ixz="0" iyy="0" iyz="0" izz="0"/>
@@ -205,14 +205,14 @@
 	<link name="cover">
 		<visual>
-			<origin xyz="['-0.01688', '-0.08366', '-0.06189']" rpy="['-3.14159', '-0.0', '0.0']"/>
+			<origin xyz="-0.01688 -0.08366 -0.06189" rpy="-3.14159 -0.0 0.0"/>
 			<geometry>
 				<mesh filename="package://sphere_description/meshes/cover.stl"/>
 			</geometry>
 			<material name="cover_material">
-				<color rgba="['0.61569', '0.81176', '0.92941', '1.0']"/>
-			</material>
-		</visual>
-		<collision>
-			<origin xyz="['-0.01688', '-0.08366', '-0.06189']" rpy="['-3.14159', '-0.0', '0.0']"/>
+				<color rgba="0.61569 0.81176 0.92941 1.0"/>
+			</material>
+		</visual>
+		<collision>
+			<origin xyz="-0.01688 -0.08366 -0.06189" rpy="-3.14159 -0.0 0.0"/>
 			<geometry>
 				<mesh filename="package://sphere_description/meshes/cover.stl"/>
@@ -220,5 +220,5 @@
 		</collision>
 		<inertial>
-			<origin xyz="['0.0', '0.0', '0.0']" rpy="['0.0', '0.0', '0.0']"/>
+			<origin xyz="0.0 0.0 0.0" rpy="0.0 0.0 0.0"/>
 			<mass value="0"/>
 			<inertia ixx="0" ixy="0" ixz="0" iyy="0" iyz="0" izz="0"/>
@@ -227,14 +227,14 @@
 	<link name="box">
 		<visual>
-			<origin xyz="['0.07606', '0.0247', '-0.0595']" rpy="['-3.14159', '-0.0', '0.0']"/>
+			<origin xyz="0.07606 0.0247 -0.0595" rpy="-3.14159 -0.0 0.0"/>
 			<geometry>
 				<mesh filename="package://sphere_description/meshes/box.stl"/>
 			</geometry>
 			<material name="box_material">
-				<color rgba="['0.61569', '0.81176', '0.92941', '1.0']"/>
-			</material>
-		</visual>
-		<collision>
-			<origin xyz="['0.07606', '0.0247', '-0.0595']" rpy="['-3.14159', '-0.0', '0.0']"/>
+				<color rgba="0.61569 0.81176 0.92941 1.0"/>
+			</material>
+		</visual>
+		<collision>
+			<origin xyz="0.07606 0.0247 -0.0595" rpy="-3.14159 -0.0 0.0"/>
 			<geometry>
 				<mesh filename="package://sphere_description/meshes/box.stl"/>
@@ -242,5 +242,5 @@
 		</collision>
 		<inertial>
-			<origin xyz="['0.0', '0.0', '0.0']" rpy="['0.0', '0.0', '0.0']"/>
+			<origin xyz="0.0 0.0 0.0" rpy="0.0 0.0 0.0"/>
 			<mass value="0"/>
 			<inertia ixx="0" ixy="0" ixz="0" iyy="0" iyz="0" izz="0"/>
@@ -249,5 +249,5 @@
 	<link name="dps310">
 		<inertial>
-			<origin xyz="['0.0', '0.0', '0.0']" rpy="['0.0', '0.0', '0.0']"/>
+			<origin xyz="0.0 0.0 0.0" rpy="0.0 0.0 0.0"/>
 			<mass value="0"/>
 			<inertia ixx="0" ixy="0" ixz="0" iyy="0" iyz="0" izz="0"/>
@@ -255,22 +255,22 @@
 	</link>
 	<joint name="dps310_frame" type="fixed">
-		<origin xyz="['0.06102', '0.06802', '-0.01803']" rpy="['-1.5708', '0.0', '0.7854']"/>
+		<origin xyz="0.06102 0.06802 -0.01803" rpy="-1.5708 0.0 0.7854"/>
 		<parent link="box"/>
 		<child link="dps310"/>
-		<axis xyz="['0.0', '0.0', '0.0']"/>
+		<axis xyz="0.0 0.0 0.0"/>
 	</joint>
 	<joint name="box_rpi_cover" type="fixed">
-		<origin xyz="['-0.09295', '-0.10836', '-0.00239']" rpy="['0.0', '-0.0', '-0.0']"/>
+		<origin xyz="-0.09295 -0.10836 -0.00239" rpy="0.0 -0.0 -0.0"/>
 		<parent link="cover"/>
 		<child link="box"/>
-		<axis xyz="['0.0', '0.0', '1.0']"/>
+		<axis xyz="0.0 0.0 1.0"/>
 		<limit effort="1" velocity="20"/>
 		<joint_properties friction="0.0"/>
 	</joint>
 	<joint name="box_rpi" type="fixed">
-		<origin xyz="['0.05801', '0.08377', '-0.06869']" rpy="['-3.14159', '0.0', '-3.14159']"/>
+		<origin xyz="0.05801 0.08377 -0.06869" rpy="-3.14159 0.0 -3.14159"/>
 		<parent link="top_bottom_mount"/>
 		<child link="cover"/>
-		<axis xyz="['0.0', '0.0', '1.0']"/>
+		<axis xyz="0.0 0.0 1.0"/>
 		<limit effort="1" velocity="20"/>
 		<joint_properties friction="0.0"/>
@@ -278,14 +278,14 @@
 	<link name="extrusions_bottom">
 		<visual>
-			<origin xyz="['-0.0', '0.18', '0.07467']" rpy="['0.0', '-0.0', '-0.0']"/>
+			<origin xyz="-0.0 0.18 0.07467" rpy="0.0 -0.0 -0.0"/>
 			<geometry>
 				<mesh filename="package://sphere_description/meshes/extrusions_bottom.stl"/>
 			</geometry>
 			<material name="extrusions_bottom_material">
-				<color rgba="['0.75294', '0.75294', '0.75294', '1.0']"/>
-			</material>
-		</visual>
-		<collision>
-			<origin xyz="['-0.0', '0.18', '0.07467']" rpy="['0.0', '-0.0', '-0.0']"/>
+				<color rgba="0.75294 0.75294 0.75294 1.0"/>
+			</material>
+		</visual>
+		<collision>
+			<origin xyz="-0.0 0.18 0.07467" rpy="0.0 -0.0 -0.0"/>
 			<geometry>
 				<mesh filename="package://sphere_description/meshes/extrusions_bottom.stl"/>
@@ -293,5 +293,5 @@
 		</collision>
 		<inertial>
-			<origin xyz="['0.0', '0.0', '0.0']" rpy="['0.0', '0.0', '0.0']"/>
+			<origin xyz="0.0 0.0 0.0" rpy="0.0 0.0 0.0"/>
 			<mass value="0"/>
 			<inertia ixx="0" ixy="0" ixz="0" iyy="0" iyz="0" izz="0"/>
@@ -300,14 +300,14 @@
 	<link name="extrusions_top">
 		<visual>
-			<origin xyz="['0.2', '-0.2', '0.0']" rpy="['3.14159', '-0.0', '0.0']"/>
+			<origin xyz="0.2 -0.2 0.0" rpy="3.14159 -0.0 0.0"/>
 			<geometry>
 				<mesh filename="package://sphere_description/meshes/extrusions_top.stl"/>
 			</geometry>
 			<material name="extrusions_top_material">
-				<color rgba="['0.75294', '0.75294', '0.75294', '1.0']"/>
-			</material>
-		</visual>
-		<collision>
-			<origin xyz="['0.2', '-0.2', '0.0']" rpy="['3.14159', '-0.0', '0.0']"/>
+				<color rgba="0.75294 0.75294 0.75294 1.0"/>
+			</material>
+		</visual>
+		<collision>
+			<origin xyz="0.2 -0.2 0.0" rpy="3.14159 -0.0 0.0"/>
 			<geometry>
 				<mesh filename="package://sphere_description/meshes/extrusions_top.stl"/>
@@ -315,5 +315,5 @@
 		</collision>
 		<inertial>
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
Commit message: Fixed all TFs, but vn100 translation under plate.

File: urdf/sphere.urdf.xacro (robot description, xacro)
@@ -52,5 +52,5 @@
 	</link>
 	<joint name="mti30_frame" type="fixed">
-		<origin xyz="-0.03005 0.00538 0.01431" rpy="-0.0 -0.0 0.7854"/>
+		<origin xyz="-0.03005 0.00538 0.01431" rpy="-0.0 -0.0 2.3562"/>
 		<parent link="mti30_body"/>
 		<child link="mti30"/>
@@ -117,5 +117,5 @@
 	</link>
 	<joint name="vn100_frame" type="fixed">
-		<origin xyz="0.00697 -0.01165 0.0012" rpy="0.0 -0.0 1.5708"/>
+		<origin xyz="0.00697 -0.01165 0.0012" rpy="3.14159 -0.0 0.0"/>
 		<parent link="vn100_lid"/>
 		<child link="vn100"/>
@@ -174,5 +174,5 @@
 	</joint>
 	<joint name="rslidar16_base_joint" type="fixed">
-		<origin xyz="0.0 -0.0 0.0068" rpy="-0.0 -0.0 2.79253"/>
+		<origin xyz="0.0 -0.0 0.0068" rpy="-0.0 -0.0 -1.91986"/>
 		<parent link="base_link"/>
 		<child link="rslidar16_body"/>

Commit message: Update meshes from Onshape after Simon's urdf fix

File: urdf/sphere.urdf.xacro (robot description, xacro)
@@ -52,5 +52,5 @@
 	</link>
 	<joint name="mti30_frame" type="fixed">
-		<origin xyz="-0.03005 0.00538 0.01431" rpy="-0.0 -0.0 2.3562"/>
+		<origin xyz="-0.03005 0.00538 0.01431" rpy="-0.0 -0.0 2.35619"/>
 		<parent link="mti30_body"/>
 		<child link="mti30"/>
@@ -117,5 +117,5 @@
 	</link>
 	<joint name="vn100_frame" type="fixed">
-		<origin xyz="0.00697 -0.01165 0.0012" rpy="3.14159 -0.0 0.0"/>
+		<origin xyz="0.00697 -0.01165 0.0012" rpy="0.0 -0.0 -3.14159"/>
 		<parent link="vn100_lid"/>
 		<child link="vn100"/>
@@ -131,5 +131,5 @@
 	</joint>
 	<joint name="vectornav_base_joint" type="fixed">
-		<origin xyz="0.0571 -0.04925 0.0068" rpy="0.0 -0.0 0.0"/>
+		<origin xyz="0.08794 -0.04925 0.0" rpy="3.14159 -0.0 3.14159"/>
 		<parent link="base_link"/>
 		<child link="vn100_base"/>
@@ -168,5 +168,5 @@
 	</link>
 	<joint name="rslidar16_frame" type="fixed">
-		<origin xyz="0.0 0.0 0.0398" rpy="0.0 0.0 0.0"/>
+		<origin xyz="0.0 0.0 0.0398" rpy="-0.0 -0.0 1.5708"/>
 		<parent link="rslidar16_body"/>
 		<child link="rslidar16"/>
@@ -174,5 +174,5 @@
 	</joint>
 	<joint name="rslidar16_base_joint" type="fixed">
-		<origin xyz="0.0 -0.0 0.0068" rpy="-0.0 -0.0 -1.91986"/>
+		<origin xyz="0.0 -0.0 0.0068" rpy="-0.0 -0.0 2.79253"/>
 		<parent link="base_link"/>
 		<child link="rslidar16_body"/>
@@ -298,34 +298,4 @@
 		</inertial>
 	</link>
-	<link name="extrusions_top">
-		<visual>
-			<origin xyz="0.2 -0.2 0.0" rpy="3.14159 -0.0 0.0"/>
-			<geometry>
-				<mesh filename="package://sphere_description/meshes/extrusions_top.stl"/>
-			</geometry>
-			<material name="extrusions_top_material">
-				<color rgba="0.75294 0.75294 0.75294 1.0"/>
-			</material>
-		</visual>
-		<collision>
-			<origin xyz="0.2 -0.2 0.0" rpy="3.14159 -0.0 0.0"/>
-			<geometry>
-				<mesh filename="package://sphere_description/meshes/extrusions_top.stl"/>
-			</geometry>
-		</collision>
-		<inertial>
-			<origin xyz="0.0 0.0 0.0" rpy="0.0 0.0 0.0"/>
-			<mass value="0"/>
-			<inertia ixx="0" ixy="0" ixz="0" iyy="0" iyz="0" izz="0"/>
-		</inertial>
-	</link>
-	<joint name="extrusions_top" type="fixed">
-		<origin xyz="-0.2 -0.02 0.07467" rpy="-3.14159 -0.0 -0.0"/>
-		<parent link="extrusions_bottom"/>
-		<child link="extrusions_top"/>
-		<axis xyz="0.0 0.0 1.0"/>
-		<limit effort="1" velocity="20"/>
-		<joint_properties friction="0.0"/>
-	</joint>
 	<link name="eyebolt">
 		<visual>

Commit message: Added the dps310 frame as measured by Nic.

File: urdf/sphere.urdf.xacro (robot description, xacro)
@@ -247,17 +247,4 @@
 		</inertial>
 	</link>
-	<link name="dps310">
-		<inertial>
-			<origin xyz="0.0 0.0 0.0" rpy="0.0 0.0 0.0"/>
-			<mass value="0"/>
-			<inertia ixx="0" ixy="0" ixz="0" iyy="0" iyz="0" izz="0"/>
-		</inertial>
-	</link>
-	<joint name="dps310_frame" type="fixed">
-		<origin xyz="0.06102 0.06802 -0.01803" rpy="-1.5708 0.0 0.7854"/>
-		<parent link="box"/>
-		<child link="dps310"/>
-		<axis xyz="0.0 0.0 0.0"/>
-	</joint>
 	<joint name="box_rpi_cover" type="fixed">
 		<origin xyz="-0.09295 -0.10836 -0.00239" rpy="0.0 -0.0 -0.0"/>
@@ -434,3 +421,9 @@
 		<joint_properties friction="0.0"/>
 	</joint>
+    <link name="dps310" />
+    <joint name="dps310_frame" type="fixed">
+        <origin xyz="0.034955 -0.040486 -0.09265" rpy="0 0 0" />
+        <parent link="rslidar16" />
+        <child link="dps310" />
+    </joint>
 </robot>
